File: PCB/GPS-Audio_PCB/_autosave-GPS-Audio_PCB.kicad_pcb (KiCad board)
At the start: 2 copper layers, 62.1 x 45.1 mm, 4 parts, among them SW1 SW_Push

Commit message: Netlify Probs
Parts:
- moved SW1 7.59 mm to (158.9, 140.5), turned to 90 degrees
Connections:
- ESP32_S1 pad RX: (no net) -> GPS TX
- ESP32_S1 pad TX: (no net) -> GPS RX
Routing:
- net GND: track 0.00 -> 40.6 mm
- net +3V3: track 0.00 -> 36.4 mm
- net GPS TX: track 0.00 -> 28.5 mm
- net GPS RX: track 0.00 -> 16.1 mm
Changed lines of the file:
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@@
 			(layers "*.Cu" "*.Mask")
 			(remove_unused_layers no)
+			(net 5 "GPS TX")
 			(thermal_bridge_angle 45)
 		)
@@
 			(layers "*.Cu" "*.Mask")
 			(remove_unused_layers no)
+			(net 6 "GPS RX")
 			(thermal_bridge_angle 45)
 		)
@@
 	(footprint "Button_Switch_THT:SW_TH_Tactile_Omron_B3F-100x"
 		(layer "F.Cu")
-		(at 163.5 134.475 -90)
+		(at 158.925 140.525 90)
 		(descr "Tactile switch, 6x6 mm, H4.3 mm, 6.5 mm pitch, https://omronfs.omron.com/en_US/ecb/products/pdf/en-b3f.pdf")
 		(tags "Omron B3F-10xx SPST 1P1T")
@@
 		)
 		(property "Datasheet" "~"
-			(at 0 0 270)
+			(at 0 0 90)
 			(unlocked yes)
 			(layer "F.Fab")
@@
 		)
 		(property "Description" "Push button switch, generic, two pins"
-			(at 0 0 270)
+			(at 0 0 90)
 			(unlocked yes)
 			(layer "F.Fab")
@@
 		(attr through_hole)
 		(fp_line
+			(start 0.75 -0.87)
+			(end 5.75 -0.87)
+			(stroke
+				(width 0.12)
+				(type solid)
+			)
+			(layer "F.SilkS")
+		)
+		(fp_line
+			(start 6.37 1.15)
+			(end 6.37 3.35)
+			(stroke
+				(width 0.12)
+				(type solid)
+			)
+			(layer "F.SilkS")
+		)
+		(fp_line
+			(start 0.13 3.35)
+			(end 0.13 1.15)
+			(stroke
+				(width 0.12)
+				(type solid)
+			)
+			(layer "F.SilkS")
+		)
+		(fp_line
 			(start 0.75 5.37)
 			(end 5.75 5.37)
-			(stroke
-				(width 0.12)
-				(type solid)
-			)
-			(layer "F.SilkS")
-		)
-		(fp_line
-			(start 0.13 3.35)
-			(end 0.13 1.15)
-			(stroke
-				(width 0.12)
-				(type solid)
-			)
-			(layer "F.SilkS")
-		)
-		(fp_line
-			(start 6.37 1.15)
-			(end 6.37 3.35)
-			(stroke
-				(width 0.12)
-				(type solid)
-			)
-			(layer "F.SilkS")
-		)
-		(fp_line
-			(start 0.75 -0.87)
-			(end 5.75 -0.87)
 			(stroke
 				(width 0.12)
@@
 		)
 		(fp_line
+			(start -1.1 -1.1)
+			(end 7.6 -1.1)
+			(stroke
+				(width 0.05)
+				(type solid)
+			)
+			(layer "F.CrtYd")
+		)
+		(fp_line
+			(start -1.1 -1.1)
+			(end -1.1 5.6)
+			(stroke
+				(width 0.05)
+				(type solid)
+			)
+			(layer "F.CrtYd")
+		)
+		(fp_line
+			(start 7.6 5.6)
+			(end 7.6 -1.1)
+			(stroke
+				(width 0.05)
+				(type solid)
+			)
+			(layer "F.CrtYd")
+		)
+		(fp_line
 			(start -1.1 5.6)
 			(end 7.6 5.6)
@@
 		)
 		(fp_line
-			(start 7.6 5.6)
-			(end 7.6 -1.1)
-			(stroke
-				(width 0.05)
-				(type solid)
-			)
-			(layer "F.CrtYd")
-		)
-		(fp_line
-			(start -1.1 -1.1)
-			(end -1.1 5.6)
-			(stroke
-				(width 0.05)
-				(type solid)
-			)
-			(layer "F.CrtYd")
-		)
-		(fp_line
-			(start -1.1 -1.1)
-			(end 7.6 -1.1)
-			(stroke
-				(width 0.05)
-				(type solid)
-			)
-			(layer "F.CrtYd")
+			(start 6.25 -0.75)
+			(end 6.25 5.25)
+			(stroke
+				(width 0.1)
+				(type solid)
+			)
+			(layer "F.Fab")
+		)
+		(fp_line
+			(start 0.25 -0.75)
+			(end 6.25 -0.75)
+			(stroke
+				(width 0.1)
+				(type solid)
+			)
+			(layer "F.Fab")
+		)
+		(fp_line
+			(start 0.25 -0.75)
+			(end 0.25 5.25)
+			(stroke
+				(width 0.1)
+				(type solid)
+			)
+			(layer "F.Fab")
 		)
 		(fp_line
@@
 			(layer "F.Fab")
 		)
-		(fp_line
-			(start 0.25 -0.75)
-			(end 0.25 5.25)
-			(stroke
-				(width 0.1)
-				(type solid)
-			)
-			(layer "F.Fab")
-		)
-		(fp_line
-			(start 0.25 -0.75)
-			(end 6.25 -0.75)
-			(stroke
-				(width 0.1)
-				(type solid)
-			)
-			(layer "F.Fab")
-		)
-		(fp_line
-			(start 6.25 -0.75)
-			(end 6.25 5.25)
-			(stroke
-				(width 0.1)
-				(type solid)
-			)
-			(layer "F.Fab")
-		)
 		(fp_text user "${REFERENCE}"
 			(at 3.25 2.25 90)
@@
 		)
 		(pad "1" thru_hole oval
-			(at 0 0 270)
+			(at 0 0 90)
 			(size 2.54 2.2)
 			(drill 0.8)
@@
 		)
 		(pad "1" thru_hole oval
-			(at 6.5 0 270)
+			(at 6.5 0 90)
 			(size 2.54 2.2)
 			(drill 0.8)
@@
 		)
 		(pad "2" thru_hole oval
-			(at 0 4.5 270)
+			(at 0 4.5 90)
 			(size 2.54 2.2)
 			(drill 0.8)
@@
 		)
 		(pad "2" thru_hole oval
-			(at 6.5 4.5 270)
+			(at 6.5 4.5 90)
 			(size 2.54 2.2)
 			(drill 0.8)
@@
 		(layer "Edge.Cuts")
 	)
+	(segment
+		(start 158.925 134.025)
+		(end 156.55 136.4)
+		(width 1)
+		(layer "B.Cu")
+		(net 1)
+	)
+	(segment
+		(start 143.157 113.568)
+		(end 142.657 113.568)
+		(width 1)
+		(layer "B.Cu")
+		(net 1)
+	)
+	(segment
+		(start 139.55 128.85)
+		(end 147.1 136.4)
+		(width 1)
+		(layer "B.Cu")
+		(net 1)
+	)
+	(segment
+		(start 156.55 136.4)
+		(end 149.2 136.4)
+		(width 1)
+		(layer "B.Cu")
+		(net 1)
+	)
+	(segment
+		(start 142.657 113.568)
+		(end 139.55 116.675)
+		(width 1)
+		(layer "B.Cu")
+		(net 1)
+	)
+	(segment
+		(start 139.55 116.675)
+		(end 139.55 128.85)
+		(width 1)
+		(layer "B.Cu")
+		(net 1)
+	)
+	(segment
+		(start 147.1 136.4)
+		(end 149.2 136.4)
+		(width 1)
+		(layer "B.Cu")
+		(net 1)
+	)
+	(segment
+		(start 143.157 110.718)
+		(end 142.682 110.718)
+		(width 1)
+		(layer "B.Cu")
+		(net 2)
+	)
+	(segment
+		(start 138.075 129.9)
+		(end 147.075 138.9)
+		(width 1)
+		(layer "B.Cu")
+		(net 2)
+	)
+	(segment
+		(start 147.075 138.9)
+		(end 149.2 138.9)
+		(width 1)
+		(layer "B.Cu")
+		(net 2)
+	)
+	(segment
+		(start 142.682 110.718)
+		(end 138.075 115.325)
+		(width 1)
+		(layer "B.Cu")
+		(net 2)
+	)
+	(segment
+		(start 138.075 115.325)
+		(end 138.075 129.9)
+		(width 1)
+		(layer "B.Cu")
+		(net 2)
+	)
+	(segment
+		(start 146.65 121.625)
+		(end 146.65 110.45)
+		(width 1)
+		(layer "B.Cu")
+		(net 5)
+	)
+	(segment
+		(start 141.95 123.35)
+		(end 144.925 123.35)
+		(width 1)
+		(layer "B.Cu")
+		(net 5)
+	)
+	(segment
+		(start 143.157 116.108)
+		(end 142.367 116.108)
+		(width 1)
+		(layer "B.Cu")
+		(net 5)
+	)
+	(segment
+		(start 140.925 122.325)
+		(end 141.95 123.35)
+		(width 1)
+		(layer "B.Cu")
+		(net 5)
+	)
+	(segment
+		(start 146.65 110.45)
+		(end 148.145 108.955)
+		(width 1)
+		(layer "B.Cu")
+		(net 5)
+	)
+	(segment
+		(start 142.367 116.108)
+		(end 140.925 117.55)
+		(width 1)
+		(layer "B.Cu")
+		(net 5)
+	)
+	(segment
+		(start 144.925 123.35)
+		(end 146.65 121.625)
+		(width 1)
+		(layer "B.Cu")
+		(net 5)
+	)
+	(segment
+		(start 140.925 117.55)
+		(end 140.925 122.325)
+		(width 1)
+		(layer "B.Cu")
+		(net 5)
+	)
+	(segment
+		(start 148.145 108.955)
+		(end 148.92 108.955)
+		(width 1)
+		(layer "B.Cu")
+		(net 5)
+	)
+	(segment
+		(start 146.65 106.415)
+		(end 148.92 106.415)
+		(width 1)
+		(layer "B.Cu")
+		(net 6)
+	)
+	(segment
+		(start 145.275 116.742)
+		(end 145.275 107.79)
+		(width 1)
+		(layer "B.Cu")
+		(net 6)
+	)
+	(segment
+		(start 143.369 118.648)
+		(end 145.275 116.742)
+		(width 1)
+		(layer "B.Cu")
+		(net 6)
+	)
+	(segment
+		(start 145.275 107.79)
+		(end 146.65 106.415)
+		(width 1)
+		(layer "B.Cu")
+		(net 6)
+	)
+	(segment
+		(start 143.157 118.648)
+		(end 143.369 118.648)
+		(width 1)
+		(layer "B.Cu")
+		(net 6)
+	)
 	(embedded_fonts no)
