File: PCB/GPS-Audio_PCB/GPS-Audio_PCB.kicad_pcb (KiCad board)
At the start: 2 copper layers, 62.1 x 45.1 mm, 4 parts, among them SW1 SW_Push

Commit message: Added some PCB Files
Parts:
- added ?: , , F.Cu at (159.2, 106.6)
- added ?: , , F.Cu at (153.8, 106.5)
- moved SW1 7.59 mm to (158.9, 140.5), turned to 90 degrees
Connections:
- ESP32_S1 pad 3V3: (no net) -> +3V3
- ESP32_S1 pad 4: (no net) -> MIC
- ESP32_S1 pad 5: (no net) -> Net-(ESP32_S1-5)
- ESP32_S1 pad GND: (no net) -> GND
- ESP32_S1 pad RX: (no net) -> GPS TX
- ESP32_S1 pad TX: (no net) -> GPS RX
Routing:
- net GND: track 0.00 -> 123.7 mm
- net +3V3: track 0.00 -> 64.9 mm
- net MIC: track 0.00 -> 45.2 mm
- net GPS TX: track 0.00 -> 28.5 mm
- net Net-(ESP32_S1-5): track 0.00 -> 19.6 mm
- net GPS RX: track 0.00 -> 16.1 mm
Other:
- board size 62.1 x 45.1 mm -> 58 x 45.2 mm
